File: hidroponik.kicad_sch (KiCad schematic)
At the start: 14 parts, among them J1 Barrel_Jack, J2 LM2596_IN, J3 ESP32_Right, J4 DS18B20_Waterproof, J5 DHT22_TempHumidity, J6 pH_Sensor_Module, J7 TDS_Sensor_Module, J8 ESP32_LEFT, J9 LM2596_OUT

Commit message: feat: add pin for ultrasonik
Parts:
- added J10: HC-SR04, Connector_PinHeader_2.54mm:PinHeader_1x04_P2.54mm_Vertical, symbol Connector_Generic:Conn_01x04
- added R4: 1k, Resistor_THT:R_Axial_DIN0207_L6.3mm_D2.5mm_P10.16mm_Horizontal, symbol Device:R
- added R5: 2k, Resistor_THT:R_Axial_DIN0207_L6.3mm_D2.5mm_P10.16mm_Horizontal, symbol Device:R
Connections:
- net +5V: now also J10.1 (Pin_1)
- net GND: now also J10.4 (Pin_4), R5.2
- net TRIG: now reaches J8.11 (Pin_11)
- net TRIG: now also J10.2 (Pin_2)
- net ECHO_ESP32: now reaches J8.13 (Pin_13)
- net ECHO_ESP32: now also R4.1, R5.1
- new net ECHO_RAW: J10.3 (Pin_3), R4.2
- no-connect marks 22 -> 20
